File: Design/H3BR20.sch (EAGLE design)
At the start: 46 parts, among them P1 HEXABIT_17.32, Q4 MMBT3904LT1, Q7 MMBT3904LT1, U1 STM32G0B1CEU6N, X1 XTALL_CSTCE8M00G52

Commit message: -Correcting some documentaion issues
Other:
- note added: "VDD = 3.3 Volts"
Changed lines of the file:
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@@
 <?xml version="1.0" encoding="utf-8"?>
 <!DOCTYPE eagle SYSTEM "eagle.dtd">
-<eagle version="9.6.1">
+<eagle version="9.6.2">
 <drawing>
 <settings>
@@
 <text x="182.7442" y="4.5992" size="1.9304" layer="101" font="vector">Ibrahim Zaeiter</text>
 <text x="254.635" y="142.24" size="1.778" layer="95">BOOT</text>
+<text x="34.925" y="199.39" size="1.778" layer="102">VDD = 3.3 Volts</text>
 </plain>
 <instances>
